Commit message: working on cpm sim

File: ROM_Rehab_Control/MATLAB_scripts/ROM_bot.urdf (robot description, URDF)
Before this commit: robot ROM_bot, 3 links, 2 joints
Links:
- link base_link: mass 0.0 -> 0.5
- link handle: mass 0.0 -> 0.1
- link lever_arm: mass 0.0 -> 0.5

Commit message: Updated RomBot class

File: ROM_Rehab_Control/MATLAB_scripts/ROM_bot.urdf (robot description, URDF)
Before this commit: robot ROM_bot, 3 links, 2 joints
Links:
- added link linear_arm, mass 0.1; visual cylinder length=0.2 radius=0.02
- link lever_arm: geometry visual cylinder length=0.2 radius=0.02
Joints:
- added joint lever_arm__linear_arm: type prismatic, parent lever_arm, child linear_arm, origin xyz=0.03 0.18 0 rpy=1.57 0 1.57, limit lower=-0.38 upper=0 effort=1000.0 velocity=0.5
- joint lever_arm__handle: origin xyz=0.03 0.4 0 rpy=0 0 0 -> xyz=0.2 0.0 0.0 rpy=0 0 0; parent lever_arm -> linear_arm
